Commit message: Quadrotor on wheels test

File: hector_quadrotor_description/urdf/quadrotor_base.urdf.xacro (robot description, xacro)
@@ -5,4 +5,7 @@
   <!-- Main quadrotor link -->
   <xacro:macro name="quadrotor_base_macro">
+    <material name="Cyan">
+      <color rgba="0 1.0 1.0 .5"/>
+    </material>
     <link name="base_link">
       <inertial>
@@ -24,4 +27,100 @@
       </collision>
     </link>
+   <link name="additional_axel">
+     <visual>
+        <origin xyz="0 0 0" rpy="0 0 0" />
+        <geometry>
+            <cylinder radius=".01" length="1"/>
+        </geometry>
+        <material name="Cyan"/>
+     </visual>
+     <collision>
+        <origin xyz="0 0 0" rpy="0 0 0" />
+        <geometry>
+            <cylinder radius=".01" length="1"/>
+        </geometry>
+     </collision>
+     <inertial>
+      <origin xyz="0 0 0" rpy="0 0 0"/>
+      <mass value="1"/>
+      <inertia
+        ixx="1.0" ixy="0.0" ixz="0.0"
+        iyy="1.0" iyz="0.0"
+        izz="1.0"/>
+    </inertial>
+   </link>
+  <gazebo reference="additional_axel">
+     <material>Gazebo/White</material>
+  </gazebo>
+     <link name="wheel1">
+     <visual>
+        <origin xyz="0 0 0" rpy="0 0 0" />
+        <geometry>
+            <cylinder radius=".5" length=".05"/>
+        </geometry>
+        <material name="Cyan"/>
+     </visual>
+     <collision>
+        <origin xyz="0 0 0" rpy="0 0 0" />
+        <geometry>
+            <cylinder radius=".5" length=".05"/>
+        </geometry>
+     </collision>
+     <inertial>
+      <origin xyz="0 0 0" rpy="0 0 0"/>
+      <mass value="1"/>
+      <inertia
+        ixx="1.0" ixy="0.0" ixz="0.0"
+        iyy="1.0" iyz="0.0"
+        izz="1.0"/>
+    </inertial>
+   </link>
+  <gazebo reference="wheel1">
+     <material>Gazebo/Black</material>
+  </gazebo>
+     <link name="wheel2">
+     <visual>
+        <origin xyz="0 0 0" rpy="0 0 0" />
+        <geometry>
+            <cylinder radius=".5" length=".05"/>
+        </geometry>
+        <material name="Cyan"/>
+     </visual>
+     <collision>
+        <origin xyz="0 0 0" rpy="0 0 0" />
+        <geometry>
+            <cylinder radius=".5" length=".05"/>
+        </geometry>
+     </collision>
+     <inertial>
+      <origin xyz="0 0 0" rpy="0 0 0"/>
+      <mass value="1"/>
+      <inertia
+        ixx="1.0" ixy="0.0" ixz="0.0"
+        iyy="1.0" iyz="0.0"
+        izz="1.0"/>
+    </inertial>
+   </link>
+  <gazebo reference="wheel2">
+     <material>Gazebo/Black</material>
+  </gazebo>
+   <joint name="centre_axel_joint" type="fixed">
+     <origin xyz="0 0 0" rpy="${pi/2} 0 ${pi/4}"/>
+     <parent link="base_link"/>
+     <child link="additional_axel"/>
+     <axis xyz="0 1 0"/>
+   </joint>
+   <joint name="wheel1_joint" type="fixed">
+     <origin xyz="0 0 .5" rpy="0 0 0"/>
+     <parent link="additional_axel"/>
+     <child link="wheel1"/>
+     <axis xyz="0 1 0"/>
+   </joint>
+   <joint name="wheel2_joint" type="fixed">
+     <origin xyz="0 0 -0.5" rpy="0 0 0"/>
+     <parent link="additional_axel"/>
+     <child link="wheel2"/>
+     <axis xyz="0 1 0"/>
+   </joint>
     <!-- Sonar height sensor -->
     <xacro:sonar_sensor name="sonar" parent="base_link" ros_topic="sonar_height" update_rate="10" min_range="0.03" max_range="3.0" field_of_view="${40*pi/180}" ray_count="3">

Commit message: added bearings to the wheels

File: hector_quadrotor_description/urdf/quadrotor_base.urdf.xacro (robot description, xacro)
@@ -76,8 +76,8 @@
     </inertial>
    </link>
-  <gazebo reference="wheel1">
+   <gazebo reference="wheel1">
      <material>Gazebo/Black</material>
-  </gazebo>
-     <link name="wheel2">
+   </gazebo>
+   <link name="wheel2">
      <visual>
         <origin xyz="0 0 0" rpy="0 0 0" />
@@ -102,7 +102,7 @@
     </inertial>
    </link>
-  <gazebo reference="wheel2">
+   <gazebo reference="wheel2">
      <material>Gazebo/Black</material>
-  </gazebo>
+   </gazebo>
    <joint name="centre_axel_joint" type="fixed">
      <origin xyz="0 0 0" rpy="${pi/2} 0 ${pi/4}"/>
@@ -111,15 +111,17 @@
      <axis xyz="0 1 0"/>
    </joint>
-   <joint name="wheel1_joint" type="fixed">
+   <joint name="wheel1_joint" type="continuous">
      <origin xyz="0 0 .5" rpy="0 0 0"/>
      <parent link="additional_axel"/>
      <child link="wheel1"/>
-     <axis xyz="0 1 0"/>
+     <axis xyz="0 0 1"/>
+     <dynamics damping="0"/>
    </joint>
-   <joint name="wheel2_joint" type="fixed">
+   <joint name="wheel2_joint" type="continuous">
      <origin xyz="0 0 -0.5" rpy="0 0 0"/>
      <parent link="additional_axel"/>
      <child link="wheel2"/>
-     <axis xyz="0 1 0"/>
+     <axis xyz="0 0 1"/>
+     <dynamics damping="0"/>
    </joint>
     <!-- Sonar height sensor -->

Commit message: Reduce wheel mass, aligned UAV y axis with additional axis, set spawning height to 0.8 to accommodate wheels

File: hector_quadrotor_description/urdf/quadrotor_base.urdf.xacro (robot description, xacro)
@@ -43,5 +43,5 @@
      <inertial>
       <origin xyz="0 0 0" rpy="0 0 0"/>
-      <mass value="1"/>
+      <mass value="0.1"/>
       <inertia
         ixx="1.0" ixy="0.0" ixz="0.0"
@@ -69,5 +69,5 @@
      <inertial>
       <origin xyz="0 0 0" rpy="0 0 0"/>
-      <mass value="1"/>
+      <mass value="0.1"/>
       <inertia
         ixx="1.0" ixy="0.0" ixz="0.0"
@@ -95,5 +95,5 @@
      <inertial>
       <origin xyz="0 0 0" rpy="0 0 0"/>
-      <mass value="1"/>
+      <mass value="0.1"/>
       <inertia
         ixx="1.0" ixy="0.0" ixz="0.0"
@@ -106,5 +106,5 @@
    </gazebo>
    <joint name="centre_axel_joint" type="fixed">
-     <origin xyz="0 0 0" rpy="${pi/2} 0 ${pi/4}"/>
+     <origin xyz="0 0 0" rpy="${pi/2} 0 0"/>
      <parent link="base_link"/>
      <child link="additional_axel"/>

Commit message: Adding pseudo motors

File: hector_quadrotor_description/urdf/quadrotor_base.urdf.xacro (robot description, xacro)
@@ -43,9 +43,9 @@
      <inertial>
       <origin xyz="0 0 0" rpy="0 0 0"/>
-      <mass value="0.1"/>
+      <mass value="0.001"/>
       <inertia
-        ixx="1.0" ixy="0.0" ixz="0.0"
-        iyy="1.0" iyz="0.0"
-        izz="1.0"/>
+        ixx="0.01" ixy="0.0" ixz="0.0"
+        iyy="0.01" iyz="0.0"
+        izz="0.01"/>
     </inertial>
    </link>
@@ -69,9 +69,9 @@
      <inertial>
       <origin xyz="0 0 0" rpy="0 0 0"/>
-      <mass value="0.1"/>
+      <mass value="0.001"/>
       <inertia
-        ixx="1.0" ixy="0.0" ixz="0.0"
-        iyy="1.0" iyz="0.0"
-        izz="1.0"/>
+        ixx="0.01" ixy="0.0" ixz="0.0"
+        iyy="0.01" iyz="0.0"
+        izz="0.01"/>
     </inertial>
    </link>
@@ -95,9 +95,9 @@
      <inertial>
       <origin xyz="0 0 0" rpy="0 0 0"/>
-      <mass value="0.1"/>
+      <mass value="0.001"/>
       <inertia
-        ixx="1.0" ixy="0.0" ixz="0.0"
-        iyy="1.0" iyz="0.0"
-        izz="1.0"/>
+        ixx="0.01" ixy="0.0" ixz="0.0"
+        iyy="0.01" iyz="0.0"
+        izz="0.01"/>
     </inertial>
    </link>
@@ -105,4 +105,30 @@
      <material>Gazebo/Black</material>
    </gazebo>
+  <link name="motor2">
+    <visual>
+      <origin xyz="0 0 0" rpy="0 0 0"/>
+      <geometry>
+        <cylinder radius="0.1" length="0.01"/>
+      </geometry>
+    </visual>
+    <collision>
+      <origin xyz="0 0 0" rpy="0 0 0"/>
+      <geometry>
+        <cylinder radius="0.1" length="0.01"/>
+      </geometry>
+    </collision>
+    <inertial>
+      <origin xyz="0 0 0" rpy="0 0 0"/>
+      <mass value="0.0001"/>
+      <inertia
+        ixx="0.01" ixy="0.0" ixz="0.0"
+        iyy="0.01" iyz="0.0"
+        izz="0.01"
+      />
+    </inertial>
+  </link>
+  <gazebo reference="motor2">
+    <material>Gazebo/Green</material>
+  </gazebo>
    <joint name="centre_axel_joint" type="fixed">
      <origin xyz="0 0 0" rpy="${pi/2} 0 0"/>
@@ -125,4 +151,9 @@
      <dynamics damping="0"/>
    </joint>
+   <joint name="motor2_joint" type="fixed">
+    <origin xyz="0 0.015 0.3" rpy="${-pi/2} 0 0"/>
+    <parent link="additional_axel"/>
+    <child link="motor2"/>
+   </joint>
     <!-- Sonar height sensor -->
     <xacro:sonar_sensor name="sonar" parent="base_link" ros_topic="sonar_height" update_rate="10" min_range="0.03" max_range="3.0" field_of_view="${40*pi/180}" ray_count="3">

Commit message: 4 pseudo motors added

File: hector_quadrotor_description/urdf/quadrotor_base.urdf.xacro (robot description, xacro)
@@ -27,30 +27,56 @@
       </collision>
     </link>
-   <link name="additional_axel">
-     <visual>
-        <origin xyz="0 0 0" rpy="0 0 0" />
-        <geometry>
-            <cylinder radius=".01" length="1"/>
-        </geometry>
-        <material name="Cyan"/>
-     </visual>
-     <collision>
-        <origin xyz="0 0 0" rpy="0 0 0" />
-        <geometry>
-            <cylinder radius=".01" length="1"/>
-        </geometry>
-     </collision>
-     <inertial>
-      <origin xyz="0 0 0" rpy="0 0 0"/>
-      <mass value="0.001"/>
-      <inertia
-        ixx="0.01" ixy="0.0" ixz="0.0"
-        iyy="0.01" iyz="0.0"
-        izz="0.01"/>
-    </inertial>
-   </link>
-  <gazebo reference="additional_axel">
-     <material>Gazebo/White</material>
-  </gazebo>
+    <link name="additional_axel">
+      <visual>
+          <origin xyz="0 0 0" rpy="0 0 0" />
+          <geometry>
+              <cylinder radius=".01" length="1"/>
+          </geometry>
+          <material name="Cyan"/>
+      </visual>
+      <collision>
+          <origin xyz="0 0 0" rpy="0 0 0" />
+          <geometry>
+              <cylinder radius=".01" length="1"/>
+          </geometry>
+      </collision>
+      <inertial>
+        <origin xyz="0 0 0" rpy="0 0 0"/>
+        <mass value="0.001"/>
+        <inertia
+          ixx="0.01" ixy="0.0" ixz="0.0"
+          iyy="0.01" iyz="0.0"
+          izz="0.01"/>
+      </inertial>
+    </link>
+    <gazebo reference="additional_axel">
+      <material>Gazebo/White</material>
+    </gazebo>
+    <link name="forward_axel">
+      <visual>
+          <origin xyz="0 0 0" rpy="0 0 0" />
+          <geometry>
+              <cylinder radius=".01" length="1"/>
+          </geometry>
+          <material name="Cyan"/>
+      </visual>
+      <collision>
+          <origin xyz="0 0 0" rpy="0 0 0" />
+          <geometry>
+              <cylinder radius=".01" length="1"/>
+          </geometry>
+      </collision>
+      <inertial>
+        <origin xyz="0 0 0" rpy="0 0 0"/>
+        <mass value="0.001"/>
+        <inertia
+          ixx="0.01" ixy="0.0" ixz="0.0"
+          iyy="0.01" iyz="0.0"
+          izz="0.01"/>
+      </inertial>
+    </link>
+    <gazebo reference="forward_axel">
+      <material>Gazebo/White</material>
+    </gazebo>
      <link name="wheel1">
      <visual>
@@ -105,55 +131,160 @@
      <material>Gazebo/Black</material>
    </gazebo>
-  <link name="motor2">
-    <visual>
-      <origin xyz="0 0 0" rpy="0 0 0"/>
-      <geometry>
-        <cylinder radius="0.1" length="0.01"/>
-      </geometry>
-    </visual>
-    <collision>
-      <origin xyz="0 0 0" rpy="0 0 0"/>
-      <geometry>
-        <cylinder radius="0.1" length="0.01"/>
-      </geometry>
-    </collision>
-    <inertial>
-      <origin xyz="0 0 0" rpy="0 0 0"/>
-      <mass value="0.0001"/>
-      <inertia
-        ixx="0.01" ixy="0.0" ixz="0.0"
-        iyy="0.01" iyz="0.0"
-        izz="0.01"
-      />
-    </inertial>
-  </link>
-  <gazebo reference="motor2">
-    <material>Gazebo/Green</material>
-  </gazebo>
-   <joint name="centre_axel_joint" type="fixed">
-     <origin xyz="0 0 0" rpy="${pi/2} 0 0"/>
-     <parent link="base_link"/>
-     <child link="additional_axel"/>
-     <axis xyz="0 1 0"/>
-   </joint>
-   <joint name="wheel1_joint" type="continuous">
-     <origin xyz="0 0 .5" rpy="0 0 0"/>
-     <parent link="additional_axel"/>
-     <child link="wheel1"/>
-     <axis xyz="0 0 1"/>
-     <dynamics damping="0"/>
-   </joint>
-   <joint name="wheel2_joint" type="continuous">
-     <origin xyz="0 0 -0.5" rpy="0 0 0"/>
-     <parent link="additional_axel"/>
-     <child link="wheel2"/>
-     <axis xyz="0 0 1"/>
-     <dynamics damping="0"/>
-   </joint>
-   <joint name="motor2_joint" type="fixed">
-    <origin xyz="0 0.015 0.3" rpy="${-pi/2} 0 0"/>
-    <parent link="additional_axel"/>
-    <child link="motor2"/>
-   </joint>
+   <link name="motor1">
+      <visual>
+        <origin xyz="0 0 0" rpy="0 0 0"/>
+        <geometry>
+          <cylinder radius="0.1" length="0.01"/>
+        </geometry>
+      </visual>
+      <collision>
+        <origin xyz="0 0 0" rpy="0 0 0"/>
+        <geometry>
+          <cylinder radius="0.1" length="0.01"/>
+        </geometry>
+      </collision>
+      <inertial>
+        <origin xyz="0 0 0" rpy="0 0 0"/>
+        <mass value="0.0001"/>
+        <inertia
+          ixx="0.01" ixy="0.0" ixz="0.0"
+          iyy="0.01" iyz="0.0"
+          izz="0.01"
+        />
+      </inertial>
+    </link>
+    <gazebo reference="motor1">
+      <material>Gazebo/Red</material>
+    </gazebo>
+    <link name="motor2">
+      <visual>
+        <origin xyz="0 0 0" rpy="0 0 0"/>
+        <geometry>
+          <cylinder radius="0.1" length="0.01"/>
+        </geometry>
+      </visual>
+      <collision>
+        <origin xyz="0 0 0" rpy="0 0 0"/>
+        <geometry>
+          <cylinder radius="0.1" length="0.01"/>
+        </geometry>
+      </collision>
+      <inertial>
+        <origin xyz="0 0 0" rpy="0 0 0"/>
+        <mass value="0.0001"/>
+        <inertia
+          ixx="0.01" ixy="0.0" ixz="0.0"
+          iyy="0.01" iyz="0.0"
+          izz="0.01"
+        />
+      </inertial>
+    </link>
+    <gazebo reference="motor2">
+      <material>Gazebo/Green</material>
+    </gazebo>
+    <link name="motor3">
+      <visual>
+        <origin xyz="0 0 0" rpy="0 0 0"/>
+        <geometry>
+          <cylinder radius="0.1" length="0.01"/>
+        </geometry>
+      </visual>
+      <collision>
+        <origin xyz="0 0 0" rpy="0 0 0"/>
+        <geometry>
+          <cylinder radius="0.1" length="0.01"/>
+        </geometry>
+      </collision>
+      <inertial>
+        <origin xyz="0 0 0" rpy="0 0 0"/>
+        <mass value="0.0001"/>
+        <inertia
+          ixx="0.01" ixy="0.0" ixz="0.0"
+          iyy="0.01" iyz="0.0"
+          izz="0.01"
+        />
+      </inertial>
+    </link>
+    <gazebo reference="motor3">
+      <material>Gazebo/Green</material>
+    </gazebo>
+    <link name="motor4">
+      <visual>
+        <origin xyz="0 0 0" rpy="0 0 0"/>
+        <geometry>
+          <cylinder radius="0.1" length="0.01"/>
+        </geometry>
+      </visual>
+      <collision>
+        <origin xyz="0 0 0" rpy="0 0 0"/>
+        <geometry>
+          <cylinder radius="0.1" length="0.01"/>
+        </geometry>
+      </collision>
+      <inertial>
+        <origin xyz="0 0 0" rpy="0 0 0"/>
+        <mass value="0.0001"/>
+        <inertia
+          ixx="0.01" ixy="0.0" ixz="0.0"
+          iyy="0.01" iyz="0.0"
+          izz="0.01"
+        />
+      </inertial>
+    </link>
+    <gazebo reference="motor4">
+      <material>Gazebo/Green</material>
+    </gazebo>
+    <joint name="centre_axel_joint" type="fixed">
+      <origin xyz="0 0 0" rpy="${pi/2} 0 0"/>
+      <parent link="base_link"/>
+      <child link="additional_axel"/>
+    </joint>
+    <joint name="centre_faxel_joint" type="fixed">
+      <origin xyz="0 0 0" rpy="0 ${pi/2} 0"/>
+      <parent link="base_link"/>
+      <child link="forward_axel"/>
+    </joint>
+    <joint name="wheel1_joint" type="continuous">
+      <origin xyz="0 0 .5" rpy="0 0 0"/>
+      <parent link="additional_axel"/>
+      <child link="wheel1"/>
+      <axis xyz="0 0 1"/>
+      <dynamics damping="0"/>
+    </joint>
+    <joint name="wheel2_joint" type="continuous">
+      <origin xyz="0 0 -0.5" rpy="0 0 0"/>
+      <parent link="additional_axel"/>
+      <child link="wheel2"/>
+      <axis xyz="0 0 1"/>
+      <dynamics damping="0"/>
+    </joint>
+    <joint name="motor1_joint" type="revolute">
+      <origin xyz="-0.015 0 0.3" rpy="0 ${-pi/2} 0"/>
+      <parent link="forward_axel"/>
+      <child link="motor1"/>
+      <axis xyz="0 0 1"/>
+      <limit effort="1000.0" velocity="0.0" lower="0.0" upper="0.0"/>
+    </joint>
+    <joint name="motor3_joint" type="revolute">
+      <origin xyz="-0.015 0 -0.3" rpy="0 ${-pi/2} 0"/>
+      <parent link="forward_axel"/>
+      <child link="motor3"/>
+      <axis xyz="0 0 1"/>
+      <limit effort="1000.0" velocity="0.0" lower="0.0" upper="0.0"/>
+    </joint>
+    <joint name="motor2_joint" type="revolute">
+      <origin xyz="0 0.015 0.3" rpy="${-pi/2} 0 0"/>
+      <parent link="additional_axel"/>
+      <child link="motor2"/>
+      <axis xyz="0 0 1"/>
+      <limit effort="1000.0" velocity="0.0" lower="0.0" upper="0.0"/>
+    </joint>
+    <joint name="motor4_joint" type="revolute">
+      <origin xyz="0 0.015 -0.3" rpy="${-pi/2} 0 0"/>
+      <parent link="additional_axel"/>
+      <child link="motor4"/>
+      <axis xyz="0 0 1"/>
+      <limit effort="1000.0" velocity="0.0" lower="0.0" upper="0.0"/>
+    </joint>
     <!-- Sonar height sensor -->
     <xacro:sonar_sensor name="sonar" parent="base_link" ros_topic="sonar_height" update_rate="10" min_range="0.03" max_range="3.0" field_of_view="${40*pi/180}" ray_count="3">

Commit message: Changed base link of the MAV from mesh to a sphere

File: hector_quadrotor_description/urdf/quadrotor_base.urdf.xacro (robot description, xacro)
@@ -14,4 +14,5 @@
         <inertia ixx="0.01152" ixy="0.0" ixz="0.0" iyy="0.01152" iyz="0.0" izz="0.0218" />
       </inertial>
+      <!-- Changing visual and collision properties
       <visual>
         <origin xyz="0 0 0" rpy="0 0 0" />
@@ -24,4 +25,17 @@
         <geometry>
           <mesh filename="package://hector_quadrotor_description/meshes/quadrotor/quadrotor_base.stl"/>
+        </geometry>
+      </collision>
+      -->
+      <visual>
+        <origin xyz="0 0 0" rpy="0 0 0"/>
+        <geometry>
+          <sphere radius="0.2"/>
+        </geometry>
+      </visual>
+      <collision>
+        <origin xyz="0 0 0" rpy="0 0 0"/>
+        <geometry>
+          <sphere radius="0.2"/>
         </geometry>
       </collision>

Commit message: Remove sphere base_link

File: hector_quadrotor_description/urdf/quadrotor_base.urdf.xacro (robot description, xacro)
@@ -14,5 +14,4 @@
         <inertia ixx="0.01152" ixy="0.0" ixz="0.0" iyy="0.01152" iyz="0.0" izz="0.0218" />
       </inertial>
-      <!-- Changing visual and collision properties
       <visual>
         <origin xyz="0 0 0" rpy="0 0 0" />
@@ -27,17 +26,18 @@
         </geometry>
       </collision>
+      <!-- Sphere visual-collision property>
+      <visual>
+        <origin xyz="0 0 0" rpy="0 0 0"/>
+        <geometry>
+          <sphere radius="0.2"/>
+        </geometry>
+      </visual>
+      <collision>
+        <origin xyz="0 0 0" rpy="0 0 0"/>
+        <geometry>
+          <sphere radius="0.2"/>
+        </geometry>
+      </collision>
       -->
-      <visual>
-        <origin xyz="0 0 0" rpy="0 0 0"/>
-        <geometry>
-          <sphere radius="0.2"/>
-        </geometry>
-      </visual>
-      <collision>
-        <origin xyz="0 0 0" rpy="0 0 0"/>
-        <geometry>
-          <sphere radius="0.2"/>
-        </geometry>
-      </collision>
     </link>
     <link name="additional_axel">
