Commit message: Bug fix on quad URDF

File: hector_quadrotor_description/urdf/quadrotor_base_alt.urdf.xacro (robot description, xacro)
@@ -13,5 +13,5 @@
   <xacro:property name="wheel_h" value="0.05"/>
   <xacro:property name="motor_connector_rad" value="0.005"/>
-  <xacro:property name="motor_connector_h" value"0.05"/>
+  <xacro:property name="motor_connector_h" value="0.05"/>
   <xacro:property name="base_mass" value="0.5"/>
   <xacro:property name="base_inertia" value="${2*base_mass*base_radius*base_radius/5}"/>
@@ -39,11 +39,11 @@
         <origin xyz="0 0 0" rpy="0 0 0"/>
         <geometry>
-          <sphere radius="${base_radius}">
-        </geometry>
-      </visual>
-      <collision>
-        <origin xyz="0 0 0" rpy="0 0 0"/>
-        <geometry>
-          <sphere radius="${base_radius}">
+          <sphere radius="${base_radius}"/>
+        </geometry>
+      </visual>
+      <collision>
+        <origin xyz="0 0 0" rpy="0 0 0"/>
+        <geometry>
+          <sphere radius="${base_radius}"/>
         </geometry>
       </collision>
@@ -90,5 +90,5 @@
     <!-- Axis 1 to rotors -->
     <link name="motor_axel_1">
-      <vidual>
+      <visual>
         <origin xyz="0 0 0" rpy="0 0 0"/>
         <geometry>
@@ -117,5 +117,5 @@
     <!-- Axis 2 to rotors -->
     <link name="motor_axel_2">
-      <vidual>
+      <visual>
         <origin xyz="0 0 0" rpy="0 0 0"/>
         <geometry>
@@ -145,11 +145,11 @@
     <link name="motor1">
       <visual>
-        <origin=xyz="0 0 0" rpy="0 0 0"/>
-        <geometry>
-          <cylinder radius="${motor_rad}" length="${motor_h}"/>
-        </geometry>
-      </visual>
-      <collision>
-        <origin=xyz="0 0 0" rpy="0 0 0"/>
+        <origin xyz="0 0 0" rpy="0 0 0"/>
+        <geometry>
+          <cylinder radius="${motor_rad}" length="${motor_h}"/>
+        </geometry>
+      </visual>
+      <collision>
+        <origin xyz="0 0 0" rpy="0 0 0"/>
         <geometry>
           <cylinder radius="${motor_rad}" length="${motor_h}"/>
@@ -171,11 +171,11 @@
     <link name="motor2">
       <visual>
-        <origin=xyz="0 0 0" rpy="0 0 0"/>
-        <geometry>
-          <cylinder radius="${motor_rad}" length="${motor_h}"/>
-        </geometry>
-      </visual>
-      <collision>
-        <origin=xyz="0 0 0" rpy="0 0 0"/>
+        <origin xyz="0 0 0" rpy="0 0 0"/>
+        <geometry>
+          <cylinder radius="${motor_rad}" length="${motor_h}"/>
+        </geometry>
+      </visual>
+      <collision>
+        <origin xyz="0 0 0" rpy="0 0 0"/>
         <geometry>
           <cylinder radius="${motor_rad}" length="${motor_h}"/>
@@ -197,11 +197,11 @@
     <link name="motor3">
       <visual>
-        <origin=xyz="0 0 0" rpy="0 0 0"/>
-        <geometry>
-          <cylinder radius="${motor_rad}" length="${motor_h}"/>
-        </geometry>
-      </visual>
-      <collision>
-        <origin=xyz="0 0 0" rpy="0 0 0"/>
+        <origin xyz="0 0 0" rpy="0 0 0"/>
+        <geometry>
+          <cylinder radius="${motor_rad}" length="${motor_h}"/>
+        </geometry>
+      </visual>
+      <collision>
+        <origin xyz="0 0 0" rpy="0 0 0"/>
         <geometry>
           <cylinder radius="${motor_rad}" length="${motor_h}"/>
@@ -223,11 +223,11 @@
     <link name="motor4">
       <visual>
-        <origin=xyz="0 0 0" rpy="0 0 0"/>
-        <geometry>
-          <cylinder radius="${motor_rad}" length="${motor_h}"/>
-        </geometry>
-      </visual>
-      <collision>
-        <origin=xyz="0 0 0" rpy="0 0 0"/>
+        <origin xyz="0 0 0" rpy="0 0 0"/>
+        <geometry>
+          <cylinder radius="${motor_rad}" length="${motor_h}"/>
+        </geometry>
+      </visual>
+      <collision>
+        <origin xyz="0 0 0" rpy="0 0 0"/>
         <geometry>
           <cylinder radius="${motor_rad}" length="${motor_h}"/>
@@ -408,5 +408,5 @@
       <material>Gazebo/Black</material>
     </gazebo>
-    <!-- Links End>
+    <!-- Links End -->
     <!-- Joints Start-->
     <!-- Base link to wheel axel -->
@@ -423,5 +423,5 @@
     </joint>
     <!-- Base link to motor axel 2 -->
-    <joint name="base_motor_axel2_joint" type="fixed"/>
+    <joint name="base_motor_axel2_joint" type="fixed">
       <origin xyz="0 0 ${base_radius/2}" rpy="${pi/2} 0 ${pi/4}"/>
       <parent link="base_link"/>

File: hector_quadrotor_description/urdf/quadrotor_hokuyo_utm30lx.urdf.xacro (robot description, xacro)
@@ -3,5 +3,5 @@
     <xacro:property name="M_PI" value="3.1415926535897931" />
     <!-- Included URDF Files -->
-    <xacro:include filename="$(find hector_quadrotor_description)/urdf/quadrotor_base.urdf.xacro" />
+    <xacro:include filename="$(find hector_quadrotor_description)/urdf/quadrotor_base_alt.urdf.xacro" />
     <!-- Instantiate quadrotor_base_macro once (has no parameters atm) -->
     <xacro:quadrotor_base_macro />

Commit message: Bug fix 2. Quad URDF

File: hector_quadrotor_description/urdf/quadrotor_base_alt.urdf.xacro (robot description, xacro)
@@ -9,6 +9,6 @@
   <xacro:property name="motor_axel_rad" value="0.01"/>
   <xacro:property name="motor_rad" value="${size_factor/8}"/>
-  <xacro:property name="motor_h" value="0.005">
-  <xacro:property name="wheel_rad" value="${size_factor}"/>
+  <xacro:property name="motor_h" value="0.005"/>
+  <xacro:property name="wheel_rad" value="${size_factor/2}"/>
   <xacro:property name="wheel_h" value="0.05"/>
   <xacro:property name="motor_connector_rad" value="0.005"/>
@@ -23,9 +23,9 @@
   <xacro:property name="motor_axel_in_izz" value="${motor_axel_mass*motor_axel_rad*motor_axel_rad/2}"/>
   <xacro:property name="motor_mass" value="0.2"/>
-  <xacro:property name="motor_ixx" value="${(motor_mass/12)*(3*motor_rad*motor*radius + motor_h*motor_h)}"/>
+  <xacro:property name="motor_ixx" value="${(motor_mass/12)*(3*motor_rad*motor_rad + motor_h*motor_h)}"/>
   <xacro:property name="motor_izz" value="${motor_mass*motor_rad*motor_rad/2}"/>
   <xacro:property name="wheel_mass" value="0.5"/>
   <xacro:property name="wheel_ixx" value="${(wheel_mass/12)*(6*wheel_rad*wheel_rad + wheel_h*wheel_h)}"/>
-  <xacro:property name="wheel_izz" value="${wheel_mass*wheel_rad*wheel_rad}">
+  <xacro:property name="wheel_izz" value="${wheel_mass*wheel_rad*wheel_rad}"/>
   <xacro:property name="motor_connector_mass" value="0.01"/>
   <xacro:property name="motor_connector_ixx" value="${(motor_connector_mass/12)*(3*motor_connector_rad*motor_connector_rad + motor_connector_h*motor_connector_h)}"/>
@@ -93,11 +93,11 @@
         <origin xyz="0 0 0" rpy="0 0 0"/>
         <geometry>
-          <cylinder radius="${motor_axel_rad}" length="motor_axel_length"/>
-        </geometry>
-      </visual>
-      <collision>
-        <origin xyz="0 0 0" rpy="0 0 0"/>
-        <geometry>
-          <cylinder radius="${motor_axel_rad}" length="motor_axel_length"/>
+          <cylinder radius="${motor_axel_rad}" length="${motor_axel_length}"/>
+        </geometry>
+      </visual>
+      <collision>
+        <origin xyz="0 0 0" rpy="0 0 0"/>
+        <geometry>
+          <cylinder radius="${motor_axel_rad}" length="${motor_axel_length}"/>
         </geometry>
       </collision>
@@ -120,11 +120,11 @@
         <origin xyz="0 0 0" rpy="0 0 0"/>
         <geometry>
-          <cylinder radius="${motor_axel_rad}" length="motor_axel_length"/>
-        </geometry>
-      </visual>
-      <collision>
-        <origin xyz="0 0 0" rpy="0 0 0"/>
-        <geometry>
-          <cylinder radius="${motor_axel_rad}" length="motor_axel_length"/>
+          <cylinder radius="${motor_axel_rad}" length="${motor_axel_length}"/>
+        </geometry>
+      </visual>
+      <collision>
+        <origin xyz="0 0 0" rpy="0 0 0"/>
+        <geometry>
+          <cylinder radius="${motor_axel_rad}" length="${motor_axel_length}"/>
         </geometry>
       </collision>
@@ -158,4 +158,5 @@
       <inertial>
         <origin xyz="0 0 0" rpy="0 0 0"/>
+        <mass value="${motor_mass}"/>
         <inertia
           ixx="${motor_ixx}" ixy="0.0" ixz="0.0"
@@ -184,4 +185,5 @@
       <inertial>
         <origin xyz="0 0 0" rpy="0 0 0"/>
+        <mass value="${motor_mass}"/>
         <inertia
           ixx="${motor_ixx}" ixy="0.0" ixz="0.0"
@@ -210,4 +212,5 @@
       <inertial>
         <origin xyz="0 0 0" rpy="0 0 0"/>
+        <mass value="${motor_mass}"/>
         <inertia
           ixx="${motor_ixx}" ixy="0.0" ixz="0.0"
@@ -236,4 +239,5 @@
       <inertial>
         <origin xyz="0 0 0" rpy="0 0 0"/>
+        <mass value="${motor_mass}"/>
         <inertia
           ixx="${motor_ixx}" ixy="0.0" ixz="0.0"
@@ -305,11 +309,11 @@
         <origin xyz="0 0 0" rpy="0 0 0" />
         <geometry>
-          <cylinder radius="motor_connector_rad" length="motor_connector_h"/>
-        </geometry>
-      </visual>
-      <collision>
-        <origin xyz="0 0 0" rpy="0 0 0" />
-        <geometry>
-          <cylinder radius="motor_connector_rad" length="motor_connector_h"/>
+          <cylinder radius="${motor_connector_rad}" length="${motor_connector_h}"/>
+        </geometry>
+      </visual>
+      <collision>
+        <origin xyz="0 0 0" rpy="0 0 0" />
+        <geometry>
+          <cylinder radius="${motor_connector_rad}" length="${motor_connector_h}"/>
         </geometry>
       </collision>
@@ -332,11 +336,11 @@
         <origin xyz="0 0 0" rpy="0 0 0" />
         <geometry>
-          <cylinder radius="motor_connector_rad" length="motor_connector_h"/>
-        </geometry>
-      </visual>
-      <collision>
-        <origin xyz="0 0 0" rpy="0 0 0" />
-        <geometry>
-          <cylinder radius="motor_connector_rad" length="motor_connector_h"/>
+          <cylinder radius="${motor_connector_rad}" length="${motor_connector_h}"/>
+        </geometry>
+      </visual>
+      <collision>
+        <origin xyz="0 0 0" rpy="0 0 0" />
+        <geometry>
+          <cylinder radius="${motor_connector_rad}" length="${motor_connector_h}"/>
         </geometry>
       </collision>
@@ -359,11 +363,11 @@
         <origin xyz="0 0 0" rpy="0 0 0" />
         <geometry>
-          <cylinder radius="motor_connector_rad" length="motor_connector_h"/>
-        </geometry>
-      </visual>
-      <collision>
-        <origin xyz="0 0 0" rpy="0 0 0" />
-        <geometry>
-          <cylinder radius="motor_connector_rad" length="motor_connector_h"/>
+          <cylinder radius="${motor_connector_rad}" length="${motor_connector_h}"/>
+        </geometry>
+      </visual>
+      <collision>
+        <origin xyz="0 0 0" rpy="0 0 0" />
+        <geometry>
+          <cylinder radius="${motor_connector_rad}" length="${motor_connector_h}"/>
         </geometry>
       </collision>
@@ -386,11 +390,11 @@
         <origin xyz="0 0 0" rpy="0 0 0" />
         <geometry>
-          <cylinder radius="motor_connector_rad" length="motor_connector_h"/>
-        </geometry>
-      </visual>
-      <collision>
-        <origin xyz="0 0 0" rpy="0 0 0" />
-        <geometry>
-          <cylinder radius="motor_connector_rad" length="motor_connector_h"/>
+          <cylinder radius="${motor_connector_rad}" length="${motor_connector_h}"/>
+        </geometry>
+      </visual>
+      <collision>
+        <origin xyz="0 0 0" rpy="0 0 0" />
+        <geometry>
+          <cylinder radius="${motor_connector_rad}" length="${motor_connector_h}"/>
         </geometry>
       </collision>
@@ -438,5 +442,5 @@
       <origin xyz="0 0 ${-wheel_axel_length/2}" rpy="0 0 0"/>
       <parent link="wheel_axel"/>
-      <childl link="wheel2"/>
+      <child link="wheel2"/>
     </joint>
     <!-- Motor axel 1 to motor con 1 -->
@@ -448,5 +452,5 @@
     <!-- Motor axel 1 to motor con 3 -->
     <joint name="axel1_motor_con3_joint" type="fixed">
-      <origin xyz="${motor_rad-(motor_axel_length/2)}" rpy="${pi/2} 0 0"/>
+      <origin xyz="0 0 ${motor_rad-(motor_axel_length/2)}" rpy="${pi/2} 0 0"/>
       <parent link="motor_axel_1"/>
       <child link="mc3"/>
@@ -454,5 +458,5 @@
     <!-- Motor axel 2 to motor con 2 -->
     <joint name="axel2_motor_con2_joint" type="fixed">
-      <origin xyz="0 0 ${(motor_axel_length/2)-motor_rad}" rpy="${pi/2} 0 0"/>
+      <origin xyz="0 0 ${(motor_axel_length/2)-motor_rad}" rpy="${-pi/2} 0 0"/>
       <parent link="motor_axel_2"/>
       <child link="mc2"/>
@@ -460,5 +464,5 @@
     <!-- Motor axel 2 to motor con 4 -->
     <joint name="axel2_motor_con4_joint" type="fixed">
-      <origin xyz="0 0 ${motor_rad-(motor_axel_length/2)}" rpy="${pi/2} 0 0"/>
+      <origin xyz="0 0 ${motor_rad-(motor_axel_length/2)}" rpy="${-pi/2} 0 0"/>
       <parent link="motor_axel_2"/>
       <child link="mc4"/>
@@ -466,5 +470,5 @@
     <!-- Motor con 1 to motor 1 -->
     <joint name="mc1_motor1_joint" type="revolute">
-      <origin xyz="0 0 motor_connector_h/2" rpy="0 0 0"/>
+      <origin xyz="0 0 ${motor_connector_h/2}" rpy="0 0 0"/>
       <parent link="mc1"/>
       <child link="motor1"/>
@@ -473,5 +477,5 @@
     <!-- Motor con 2 to motor 2 -->
     <joint name="mc2_motor2_joint" type="revolute">
-      <origin xyz="0 0 motor_connector_h/2" rpy="0 0 0"/>
+      <origin xyz="0 0 ${motor_connector_h/2}" rpy="0 0 0"/>
       <parent link="mc2"/>
       <child link="motor2"/>
@@ -480,5 +484,5 @@
     <!-- Motor con 3 to motor 3 -->
     <joint name="mc3_motor3_joint" type="revolute">
-      <origin xyz="0 0 motor_connector_h/2" rpy="0 0 0"/>
+      <origin xyz="0 0 ${motor_connector_h/2}" rpy="0 0 0"/>
       <parent link="mc3"/>
       <child link="motor3"/>
@@ -486,8 +490,8 @@
     </joint>
     <!-- Motor con 4 to motor 4 -->
-    <joint name="mc3_motor3_joint" type="revolute">
-      <origin xyz="0 0 motor_connector_h/2" rpy="0 0 0"/>
-      <parent link="mc3"/>
-      <child link="motor3"/>
+    <joint name="mc4_motor4_joint" type="revolute">
+      <origin xyz="0 0 ${motor_connector_h/2}" rpy="0 0 0"/>
+      <parent link="mc4"/>
+      <child link="motor4"/>
       <limit effort="1000.0" velocity="0.0" lower="0.0" upper="0.0"/>
     </joint>

Commit message: Fix bug in wheel-axel joints

File: hector_quadrotor_description/urdf/quadrotor_base_alt.urdf.xacro (robot description, xacro)
@@ -437,4 +437,6 @@
       <parent link="wheel_axel"/>
       <child link="wheel1"/>
+      <axis xyz="0 0 1"/>
+      <dynamics damping="0"/>
     </joint>
     <!-- Wheel axel to wheel 2 -->
@@ -443,4 +445,6 @@
       <parent link="wheel_axel"/>
       <child link="wheel2"/>
+      <axis xyz="0 0 1"/>
+      <dynamics damping="0"/>
     </joint>
     <!-- Motor axel 1 to motor con 1 -->
